File: mitten40percentPCB/mitten40percent.kicad_sch (KiCad schematic)
At the start: 10 parts, among them SW1 SW_Push, U1 STM32F072CBT6

Commit message: stm32 wiring finally finished!!!! (theres a non-zero percent chance it will burn my house down)
Parts:
- added C10, C11: 1uF, symbol Device:C
- added C8: 100nF, symbol Device:C
- added C9: 4.7uF, symbol Device:C
- added D1, D10, D11, D12, D13, D14, D15, D16, D17, D18, D19, D2, D20, D21, D22, D23, D24, D25, D26, D27, D28, D29, D3, D30, D31, D32, D33, D34, D35, D36, D37, D38, D39, D4, D40, D41, D42, D43, D44, D45, D47, D5, D6, D7, D8, D9: D, symbol Device:D
- added F1: 500mA, symbol Device:Fuse
- added J1: USB_C_Receptacle_USB2.0_14P, symbol Connector:USB_C_Receptacle_USB2.0_14P
- added R2, R3: 5.1k, symbol Device:R
- added SW1, SW10, SW11, SW12, SW13, SW14, SW15, SW16, SW17, SW18, SW19, SW2, SW20, SW21, SW22, SW23, SW24, SW25, SW26, SW27, SW28, SW29, SW3, SW30, SW31, SW32, SW33, SW34, SW35, SW36, SW37, SW38, SW39, SW4, SW40, SW41, SW42, SW43, SW44, SW45, SW47, SW5, SW6, SW7, SW8, SW9: SW_Push_45deg, symbol Switch:SW_Push_45deg
- added SW46: RotaryEncoder_Switch, symbol Device:RotaryEncoder_Switch
- added U2: USBLC6-2SC6, Package_TO_SOT_SMD:SOT-23-6, symbol Power_Protection:USBLC6-2SC6
- added U3: XC6206PxxxMR, Package_TO_SOT_SMD:SOT-23-3, symbol Regulator_Linear:XC6206PxxxMR
- C4: value 100nF -> 4.7uF
- C6: value 100nF -> 10nF
- C7: value 10uF -> 1uF
- renumbered SW1 to SW0
Connections:
- net +3.3V: now also C11.1, C8.1, C9.1, U3.2 (VO)
- net GND: now also C10.2, C11.2, C8.2, C9.2, J1.A1 (GND), J1.A12 (GND), J1.B1 (GND), J1.B12 (GND), J1.SH (SHIELD), R2.2, R3.2, U2.2 (GND), U3.1 (GND)
- net MCU_D-: now reaches U1.32 (PA11)
- net MCU_D-: now also U2.3 (I/O2)
- net MCU_D+: now reaches U1.33 (PA12)
- net MCU_D+: now also U2.1 (I/O1)
- new net: SW19.1, SW36.1, SW37.1, SW7.1
- new net: D19.2 (A), SW19.2
- new net: SW1.1, SW13.1, SW25.1, SW26.1
- new net: D13.2 (A), SW13.2
- new net: D1.1 (K), D10.1 (K), D11.1 (K), D12.1 (K), D2.1 (K), D3.1 (K), D4.1 (K), D5.1 (K), D6.1 (K), D7.1 (K), D8.1 (K), D9.1 (K)
- new net: D5.2 (A), SW5.2
- new net: D26.1 (K), D28.1 (K), D30.1 (K), D32.1 (K), D34.1 (K), D36.1 (K), D38.1 (K), D40.1 (K), D42.1 (K), D44.1 (K)
- new net: D44.2 (A), SW44.2
- new net: SW16.1, SW31.1, SW32.1, SW4.1
- new net: D4.2 (A), SW4.2
- new net: D30.2 (A), SW30.2
- new net: D1.2 (A), SW1.2
- new net: SW20.1, SW39.1, SW8.1
- new net: D20.2 (A), SW20.2
- new net: SW10.1, SW22.1, SW40.1, SW43.1
- new net: D22.2 (A), SW22.2
- new net: D13.1 (K), D14.1 (K), D15.1 (K), D16.1 (K), D17.1 (K), D18.1 (K), D19.1 (K), D20.1 (K), D21.1 (K), D22.1 (K), D23.1 (K), D24.1 (K)
- new net: D14.2 (A), SW14.2
- new net: D24.2 (A), SW24.2
- new net: D10.2 (A), SW10.2
- new net: SW18.1, SW35.1, SW6.1
- new net: D18.2 (A), SW18.2
- new net: D28.2 (A), SW28.2
- new net: D25.1 (K), D27.1 (K), D29.1 (K), D31.1 (K), D33.1 (K), D35.1 (K), D37.1 (K), D39.1 (K), D41.1 (K), D43.1 (K), D45.1 (K), D47.1 (K)
- new net: D25.2 (A), SW25.2
- new net: D40.2 (A), SW40.2
- new net: SW15.1, SW29.1, SW3.1, SW30.1
- new net: D15.2 (A), SW15.2
- new net: D3.2 (A), SW3.2
- new net: D16.2 (A), SW16.2
- new net: SW14.1, SW2.1, SW27.1, SW28.1
- new net: D7.2 (A), SW7.2
- new net: D35.2 (A), SW35.2
- new net: SW21.1, SW38.1, SW41.1, SW9.1
- new net: D38.2 (A), SW38.2
- new net: D11.2 (A), SW11.2
- new net: D43.2 (A), SW43.2
- new net: SW12.1, SW24.1, SW44.1, SW47.1
- new net: D12.2 (A), SW12.2
- new net: D17.2 (A), SW17.2
- new net: D47.2 (A), SW47.2
- new net: D41.2 (A), SW41.2
- new net: D36.2 (A), SW36.2
- new net: D45.2 (A), SW45.2
- new net: SW11.1, SW23.1, SW42.1, SW45.1
- new net: D6.2 (A), SW6.2
- new net: D23.2 (A), SW23.2
- new net: D33.2 (A), SW33.2
- new net: SW17.1, SW33.1, SW34.1, SW5.1
- new net: D2.2 (A), SW2.2
- new net: D39.2 (A), SW39.2
- new net: D31.2 (A), SW31.2
- new net: D29.2 (A), SW29.2
- new net: D27.2 (A), SW27.2
- new net: D34.2 (A), SW34.2
- new net: D37.2 (A), SW37.2
- new net: D8.2 (A), SW8.2
- new net: D32.2 (A), SW32.2
- new net: J1.A5 (CC1), R2.1
- new net: J1.B5 (CC2), R3.1
- new net: D26.2 (A), SW26.2
- new net: D9.2 (A), SW9.2
- new net: D42.2 (A), SW42.2
- new net: D21.2 (A), SW21.2
- new net +5V: C10.1, F1.2, U3.3 (VI)
- new net USB_D+: J1.A6 (D+), J1.B6 (D+), U2.6 (I/O1)
- new net USB_D-: J1.A7 (D-), J1.B7 (D-), U2.4 (I/O2)
- new net VBUS: F1.1, J1.A4 (VBUS), J1.A9 (VBUS), J1.B4 (VBUS), J1.B9 (VBUS), U2.5 (VBUS)
Other:
- moved on the sheet: C1, R1, SW0, U1

Commit message: added rows and columns
Connections:
- net C6: now reaches SW19.1, SW36.1, SW37.1, SW7.1
- net C6: now also U1.42 (PB6)
- net C0: now reaches SW1.1, SW13.1, SW25.1, SW26.1
- net C0: now also U1.18 (PB0)
- net R0: now reaches D1.1 (K), D10.1 (K), D11.1 (K), D12.1 (K), D2.1 (K), D3.1 (K), D4.1 (K), D5.1 (K), D6.1 (K), D7.1 (K), D8.1 (K), D9.1 (K)
- net R0: now also U1.25 (PB12)
- net R3: now reaches D26.1 (K), D28.1 (K), D30.1 (K), D32.1 (K), D34.1 (K), D36.1 (K), D38.1 (K), D40.1 (K), D42.1 (K), D44.1 (K)
- net R3: now also U1.28 (PB15)
- net C3: now reaches SW16.1, SW31.1, SW32.1, SW4.1
- net C3: now also U1.39 (PB3)
- net C7: now reaches SW20.1, SW39.1, SW8.1
- net C7: now also U1.43 (PB7)
- net C9: now reaches SW10.1, SW22.1, SW40.1, SW43.1
- net C9: now also U1.46 (PB9)
- net R1: now reaches D13.1 (K), D14.1 (K), D15.1 (K), D16.1 (K), D17.1 (K), D18.1 (K), D19.1 (K), D20.1 (K), D21.1 (K), D22.1 (K), D23.1 (K), D24.1 (K)
- net R1: now also U1.26 (PB13)
- net C5: now reaches SW18.1, SW35.1, SW6.1
- net C5: now also U1.41 (PB5)
- net R2: now reaches D25.1 (K), D27.1 (K), D29.1 (K), D31.1 (K), D33.1 (K), D35.1 (K), D37.1 (K), D39.1 (K), D41.1 (K), D43.1 (K), D45.1 (K), D47.1 (K)
- net R2: now also U1.27 (PB14)
- net C2: now reaches SW15.1, SW29.1, SW3.1, SW30.1
- net C2: now also U1.20 (PB2)
- net C1: now reaches SW14.1, SW2.1, SW27.1, SW28.1
- net C1: now also U1.19 (PB1)
- net C8: now reaches SW21.1, SW38.1, SW41.1, SW9.1
- net C8: now also U1.45 (PB8)
- net C11: now reaches SW12.1, SW24.1, SW44.1, SW47.1
- net C11: now also U1.22 (PB11)
- net C10: now reaches SW11.1, SW23.1, SW42.1, SW45.1
- net C10: now also U1.21 (PB10)
- net C4: now reaches SW17.1, SW33.1, SW34.1, SW5.1
- net C4: now also U1.40 (PB4)
Other:
- moved on the sheet: D1, D10, D11, D12, D13, D14, D15, D16, D17, D18, D19, D2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

Commit message: completed first passthrough of schematic, implemented a joystick and a screen
Parts:
- removed D47: D, symbol Device:D
- removed J1: USB_C_Receptacle_USB2.0_14P, symbol Connector:USB_C_Receptacle_USB2.0_14P
- removed SW46: RotaryEncoder_Switch, symbol Device:RotaryEncoder_Switch
- removed SW47: SW_Push_45deg, symbol Switch:SW_Push_45deg
- added D46: D, Diode_SMD:D_SOD-123, symbol Device:D
- added J2: I2C, PCM_SparkFun-Connector:1x04_P2.54mm, symbol PCM_SparkFun-Connector:I2CStandard_1x04_P2.54mm
- added J3: USB_C_Receptacle_USB2.0_16P, Connector_USB:USB_C_Receptacle_HCTL_HC-TYPE-C-16P-01A, symbol Connector:USB_C_Receptacle_USB2.0_16P
- added SW46: SW_Push_45deg, Button_Switch_Keyboard:SW_Cherry_MX_1.00u_PCB, symbol Switch:SW_Push_45deg
- added SW48: Joystick, PCM_SparkFun-Switch:Joystick_PTH, symbol PCM_SparkFun-Switch:Joystick_PTH
- C1, C10, C11, C2, C3, C4, C5, C6, C7, C8, C9: footprint (none) -> Capacitor_SMD:C_0402_1005Metric
- D1, D10, D11, D12, D13, D14, D15, D16, D17, D18, D19, D2, D20, D21, D22, D23, D24, D25, D26, D27, D28, D29, D3, D30, D31, D32, D33, D34, D35, D36, D37, D38, D39, D4, D40, D41, D42, D43, D44, D45, D5, D6, D7, D8, D9: footprint (none) -> Diode_SMD:D_SOD-123
- F1: footprint (none) -> Fuse:Fuse_0603_1608Metric
- R1, R2, R3: footprint (none) -> Resistor_SMD:R_0402_1005Metric
- SW0: footprint (none) -> Button_Switch_SMD:SW_SPST_TL3342
- SW1, SW10, SW11, SW12, SW13, SW14, SW15, SW16, SW17, SW18, SW19, SW2, SW20, SW21, SW22, SW23, SW24, SW25, SW26, SW27, SW28, SW29, SW3, SW30, SW31, SW32, SW33, SW34, SW35, SW36, SW37, SW38, SW39, SW4, SW40, SW41, SW42, SW43, SW44, SW45, SW5, SW6, SW7, SW8, SW9: footprint (none) -> Button_Switch_Keyboard:SW_Cherry_MX_1.00u_PCB
Connections:
- net +3.3V: now also SW48.VCC
- net C0: now also SW37.1, U1.25 (PB12); no longer SW26.1, U1.18 (PB0)
- net C1: now also SW26.1, SW38.1, U1.26 (PB13); no longer SW27.1, SW28.1, U1.19 (PB1)
- net C10: now also SW35.1, U1.29 (PA8); no longer SW42.1, U1.21 (PB10)
- net C11: now also SW36.1, U1.30 (PA9), SW46.1; no longer SW44.1, U1.22 (PB11)
- net C2: now also SW27.1, SW39.1, U1.27 (PB14); no longer SW29.1, SW30.1, U1.20 (PB2)
- net C3: now also SW28.1, SW40.1, U1.28 (PB15); no longer SW31.1, SW32.1, U1.39 (PB3)
- net C4: now also SW29.1, SW41.1, U1.12 (PA2); no longer SW33.1, SW34.1, U1.40 (PB4)
- net C5: now also SW30.1, U1.13 (PA3); no longer SW35.1, U1.41 (PB5)
- net C6: now also SW31.1, SW42.1, U1.14 (PA4); no longer SW36.1, SW37.1, U1.42 (PB6)
- net C7: now also SW32.1, U1.15 (PA5); no longer SW39.1, U1.43 (PB7)
- net C8: now also SW33.1, SW43.1, U1.16 (PA6); no longer SW38.1, SW41.1, U1.45 (PB8)
- net C9: now also SW34.1, SW44.1, U1.17 (PA7); no longer SW40.1, SW43.1, U1.46 (PB9)
- net GND: now also J2.1 (Pin_1), J3.A1 (GND), J3.A12 (GND), J3.B1 (GND), J3.B12 (GND), J3.SH (SHIELD), SW48.GND
- net R0: now also U1.42 (PB6); no longer U1.25 (PB12)
- net R1: now also U1.43 (PB7); no longer U1.26 (PB13)
- net R2: now also D26.1 (K), D28.1 (K), D30.1 (K), D32.1 (K), D34.1 (K), D36.1 (K), U1.45 (PB8); no longer D37.1 (K), D39.1 (K), D41.1 (K), D43.1 (K), D45.1 (K), U1.27 (PB14)
- net R3: now also D37.1 (K), D39.1 (K), D41.1 (K), D43.1 (K), D45.1 (K), U1.46 (PB9), D46.1 (K); no longer D26.1 (K), D28.1 (K), D30.1 (K), D32.1 (K), D34.1 (K), D36.1 (K), U1.28 (PB15)
- net USB_D+: now also J3.A6 (D+), J3.B6 (D+)
- net USB_D-: now also J3.A7 (D-), J3.B7 (D-)
- net VBUS: now also J3.A4 (VBUS), J3.A9 (VBUS), J3.B4 (VBUS), J3.B9 (VBUS)
- net JoystickX: now reaches U1.34 (PA13)
- net JoystickX: now also SW48.Horizontal
- net JoystickY: now reaches U1.37 (PA14)
- net JoystickY: now also SW48.Vertical
- net JoystickSelect: now reaches U1.38 (PA15)
- net JoystickSelect: now also SW48.Select
- net at R2.1: now also J3.A5 (CC1)
- net at R3.1: now also J3.B5 (CC2)
- new net: D46.2 (A), SW46.2
- new net +3V3: J2.2 (Pin_2)
- new net SCL: J2.4 (Pin_4), U1.21 (PB10)
- new net SDA: J2.3 (Pin_3), U1.22 (PB11)
- no-connect marks 0 -> 3
Other:
- moved on the sheet: C1, U1

Commit message: implemented key layout on pcb, partially done with implementation of stm32
Parts:
- SW41, SW42: footprint Button_Switch_Keyboard:SW_Cherry_MX_1.00u_PCB -> Button_Switch_Keyboard:SW_Cherry_MX_2.00u_PCB
Changed lines of the file:
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@@
 			)
 		)
-		(property "Footprint" "Button_Switch_Keyboard:SW_Cherry_MX_1.00u_PCB"
+		(property "Footprint" "Button_Switch_Keyboard:SW_Cherry_MX_2.00u_PCB"
 			(at 167.64 95.25 0)
 			(hide yes)
@@
 			)
 		)
-		(property "Footprint" "Button_Switch_Keyboard:SW_Cherry_MX_1.00u_PCB"
+		(property "Footprint" "Button_Switch_Keyboard:SW_Cherry_MX_2.00u_PCB"
 			(at 200.66 95.25 0)
 			(hide yes)

Commit message: removed two unecessary .md files
Parts:
- J2: footprint PCM_SparkFun-Connector:1x04_P2.54mm -> Display:ER_OLEDM0.91_1x-I2C
Other:
- company: (none) -> poo poo pee pee corporation
- title: (none) -> mitten40 PCB
Changed lines of the file:
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@@
 	(generator_version "10.0")
 	(paper "A4")
+	(title_block
+		(title "mitten40 PCB")
+		(rev "0")
+		(company "poo poo pee pee corporation")
+	)
 	(junction
 		(at 257.81 105.41)
@@
 			)
 		)
-		(property "Footprint" "PCM_SparkFun-Connector:1x04_P2.54mm"
+		(property "Footprint" "Display:ER_OLEDM0.91_1x-I2C"
 			(at 31.75 135.89 0)
 			(hide yes)

Commit message: finished wiring individual components (stm32, usb-c port, reset button), routed the matrix to the mcu
Connections:
- net C0: now also U1.31 (PA10); no longer U1.25 (PB12)
- net C1: now also U1.30 (PA9); no longer U1.26 (PB13)
- net C10: now also U1.14 (PA4); no longer U1.29 (PA8)
- net C11: now also U1.13 (PA3); no longer U1.30 (PA9)
- net C2: now also U1.29 (PA8); no longer U1.27 (PB14)
- net C4: now also U1.27 (PB14); no longer U1.12 (PA2)
- net C5: now also U1.26 (PB13); no longer U1.13 (PA3)
- net C6: now also U1.25 (PB12); no longer U1.14 (PA4)
- net C7: now also U1.17 (PA7); no longer U1.15 (PA5)
- net C9: now also U1.15 (PA5); no longer U1.17 (PA7)
Changed lines of the file:
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@@
-		)
-	)
-	(label "C6"
-		(at 58.42 36.83 0)
-		(effects
-			(font
-				(size 1.27 1.27)
-			)
-			(justify left bottom)
-		)
-	)
-	(label "C12"
-		(at 71.12 148.59 270)
-		(effects
-			(font
-				(size 1.27 1.27)
-			)
-			(justify right bottom)
 		)
 	)
@@
 		)
 	)
+	(label "C0"
+		(at 58.42 52.07 0)
+		(effects
+			(font
+				(size 1.27 1.27)
+			)
+			(justify left bottom)
+		)
+	)
 	(label "R3"
 		(at 279.4 105.41 0)
@@
 		)
 	)
+	(label "C2"
+		(at 58.42 46.99 0)
+		(effects
+			(font
+				(size 1.27 1.27)
+			)
+			(justify left bottom)
+		)
+	)
 	(label "USB_D+"
 		(at 165.1 171.45 0)
@@
 		)
 	)
-	(label "C10"
-		(at 58.42 46.99 0)
-		(effects
-			(font
-				(size 1.27 1.27)
-			)
-			(justify left bottom)
-		)
-	)
 	(label "VBAT"
 		(at 35.56 19.05 90)
@@
 		)
 	)
-	(label "C4"
-		(at 58.42 31.75 0)
-		(effects
-			(font
-				(size 1.27 1.27)
-			)
-			(justify left bottom)
-		)
-	)
 	(label "SDA"
 		(at 22.86 82.55 180)
@@
 		)
 	)
+	(label "C3"
+		(at 22.86 92.71 180)
+		(effects
+			(font
+				(size 1.27 1.27)
+			)
+			(justify right bottom)
+		)
+	)
 	(label "JoystickY"
 		(at 63.5 113.03 0)
@@
 		)
 	)
+	(label "C1"
+		(at 58.42 49.53 0)
+		(effects
+			(font
+				(size 1.27 1.27)
+			)
+			(justify left bottom)
+		)
+	)
 	(label "MCU_D+"
 		(at 58.42 57.15 0)
@@
 		)
 	)
-	(label "C11"
-		(at 58.42 49.53 0)
-		(effects
-			(font
-				(size 1.27 1.27)
-			)
-			(justify left bottom)
-		)
-	)
 	(label "SCL"
 		(at 22.86 80.01 180)
@@
 		)
 	)
+	(label "C6"
+		(at 22.86 85.09 180)
+		(effects
+			(font
+				(size 1.27 1.27)
+			)
+			(justify right bottom)
+		)
+	)
+	(label "C10"
+		(at 58.42 36.83 0)
+		(effects
+			(font
+				(size 1.27 1.27)
+			)
+			(justify left bottom)
+		)
+	)
 	(label "C3"
 		(at 137.16 24.13 0)
@@
 		)
 	)
-	(label "C0"
-		(at 22.86 85.09 180)
-		(effects
-			(font
-				(size 1.27 1.27)
-			)
-			(justify right bottom)
+	(label "C4"
+		(at 22.86 90.17 180)
+		(effects
+			(font
+				(size 1.27 1.27)
+			)
+			(justify right bottom)
+		)
+	)
+	(label "C2"
+		(at 120.65 24.13 0)
+		(effects
+			(font
+				(size 1.27 1.27)
+			)
+			(justify left bottom)
+		)
+	)
+	(label "C7"
+		(at 203.2 24.13 0)
+		(effects
+			(font
+				(size 1.27 1.27)
+			)
+			(justify left bottom)
+		)
+	)
+	(label "C9"
+		(at 58.42 39.37 0)
+		(effects
+			(font
+				(size 1.27 1.27)
+			)
+			(justify left bottom)
+		)
+	)
+	(label "MCU_D+"
+		(at 57.15 180.34 180)
+		(effects
+			(font
+				(size 1.27 1.27)
+			)
+			(justify right bottom)
+		)
+	)
+	(label "BOOT0"
+		(at 22.86 31.75 180)
+		(effects
+			(font
+				(size 1.27 1.27)
+			)
+			(justify right bottom)
+		)
+	)
+	(label "R3"
+		(at 22.86 77.47 180)
+		(effects
+			(font
+				(size 1.27 1.27)
+			)
+			(justify right bottom)
+		)
+	)
+	(label "C5"
+		(at 22.86 87.63 180)
+		(effects
+			(font
+				(size 1.27 1.27)
+			)
+			(justify right bottom)
+		)
+	)
+	(label "C7"
+		(at 58.42 44.45 0)
+		(effects
+			(font
+				(size 1.27 1.27)
+			)
+			(justify left bottom)
+		)
+	)
+	(label "C9"
+		(at 236.22 24.13 0)
+		(effects
+			(font
+				(size 1.27 1.27)
+			)
+			(justify left bottom)
+		)
+	)
+	(label "R1"
+		(at 279.4 64.77 0)
+		(effects
+			(font
+				(size 1.27 1.27)
+			)
+			(justify left bottom)
 		)
 	)
@@
 		)
 	)
-	(label "C2"
-		(at 120.65 24.13 0)
-		(effects
-			(font
-				(size 1.27 1.27)
-			)
-			(justify left bottom)
-		)
-	)
-	(label "C2"
-		(at 22.86 90.17 180)
-		(effects
-			(font
-				(size 1.27 1.27)
-			)
-			(justify right bottom)
-		)
-	)
-	(label "C7"
-		(at 203.2 24.13 0)
-		(effects
-			(font
-				(size 1.27 1.27)
-			)
-			(justify left bottom)
-		)
-	)
-	(label "C9"
-		(at 58.42 44.45 0)
-		(effects
-			(font
-				(size 1.27 1.27)
-			)
-			(justify left bottom)
-		)
-	)
-	(label "MCU_D+"
-		(at 57.15 180.34 180)
-		(effects
-			(font
-				(size 1.27 1.27)
-			)
-			(justify right bottom)
-		)
-	)
-	(label "C1"
-		(at 22.86 87.63 180)
-		(effects
-			(font
-				(size 1.27 1.27)
-			)
-			(justify right bottom)
-		)
-	)
-	(label "BOOT0"
-		(at 22.86 31.75 180)
-		(effects
-			(font
-				(size 1.27 1.27)
-			)
-			(justify right bottom)
-		)
-	)
-	(label "R3"
-		(at 22.86 77.47 180)
-		(effects
-			(font
-				(size 1.27 1.27)
-			)
-			(justify right bottom)
-		)
-	)
-	(label "C7"
-		(at 58.42 39.37 0)
-		(effects
-			(font
-				(size 1.27 1.27)
-			)
-			(justify left bottom)
-		)
-	)
-	(label "C9"
-		(at 236.22 24.13 0)
-		(effects
-			(font
-				(size 1.27 1.27)
-			)
-			(justify left bottom)
-		)
-	)
-	(label "C3"
-		(at 22.86 92.71 180)
-		(effects
-			(font
-				(size 1.27 1.27)
-			)
-			(justify right bottom)
-		)
-	)
-	(label "R1"
-		(at 279.4 64.77 0)
-		(effects
-			(font
-				(size 1.27 1.27)
-			)
-			(justify left bottom)
-		)
-	)
 	(label "VDDIO2"
 		(at 45.72 19.05 90)
@@
 		)
 	)
-	(label "C5"
-		(at 58.42 34.29 0)
-		(effects
-			(font
-				(size 1.27 1.27)
-			)
-			(justify left bottom)
-		)
-	)
 	(label "SDA"
 		(at 26.67 124.46 180)
@@
 		(effects
 			(font
+				(size 1.27 1.27)
+			)
+			(justify left bottom)
+		)
+	)
+	(label "C11"
+		(at 58.42 34.29 0)
+		(effects
+			(font

Commit message: finished routing and ground fill, now on to santiy checks
Connections:
- net +3V3 is gone; now on net +3.3V: J2.2 (Pin_2)
- no-connect marks 3 -> 17
Changed lines of the file:
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@@
 	)
 	(no_connect
+		(at 22.86 39.37)
+	)
+	(no_connect
 		(at 162.56 180.34)
 	)
 	(no_connect
+		(at 22.86 36.83)
+	)
+	(no_connect
+		(at 22.86 62.23)
+	)
+	(no_connect
+		(at 22.86 67.31)
+	)
+	(no_connect
+		(at 58.42 29.21)
+	)
+	(no_connect
 		(at 162.56 182.88)
 	)
 	(no_connect
+		(at 22.86 49.53)
+	)
+	(no_connect
+		(at 22.86 46.99)
+	)
+	(no_connect
+		(at 22.86 59.69)
+	)
+	(no_connect
+		(at 58.42 26.67)
+	)
+	(no_connect
 		(at 74.93 132.08)
 	)
+	(no_connect
+		(at 22.86 54.61)
+	)
+	(no_connect
+		(at 22.86 64.77)
+	)
+	(no_connect
+		(at 22.86 57.15)
+	)
+	(no_connect
+		(at 22.86 44.45)
+	)
+	(no_connect
+		(at 58.42 31.75)
+	)
 	(wire
 		(pts
@@
 	)
 	(symbol
-		(lib_id "power:+3V3")
-		(at 19.05 127 0)
-		(unit 1)
-		(body_style 1)
-		(exclude_from_sim no)
-		(in_bom yes)
-		(on_board yes)
-		(in_pos_files yes)
-		(dnp no)
-		(fields_autoplaced yes)
-		(property "Reference" "#PWR028"
-			(at 19.05 130.81 0)
-			(hide yes)
-			(show_name no)
-			(do_not_autoplace no)
-			(effects
-				(font
-					(size 1.27 1.27)
-				)
-			)
-		)
-		(property "Value" "+3V3"
-			(at 19.05 121.92 0)
-			(show_name no)
-			(do_not_autoplace no)
-			(effects
-				(font
-					(size 1.27 1.27)
-				)
-			)
-		)
-		(property "Footprint" ""
-			(at 19.05 127 0)
-			(hide yes)
-			(show_name no)
-			(do_not_autoplace no)
-			(effects
-				(font
-					(size 1.27 1.27)
-				)
-			)
-		)
-		(property "Datasheet" ""
-			(at 19.05 127 0)
-			(hide yes)
-			(show_name no)
-			(do_not_autoplace no)
-			(effects
-				(font
-					(size 1.27 1.27)
-				)
-			)
-		)
-		(property "Description" "Power symbol creates a global label with name \"+3V3\""
-			(at 19.05 127 0)
-			(hide yes)
-			(show_name no)
-			(do_not_autoplace no)
-			(effects
-				(font
-					(size 1.27 1.27)
-				)
-			)
-		)
-		(pin "1"
-		)
-		(instances
-			(project "mitten40percent"
-				(path "/4d97bcd4-b797-40db-b476-9202db9dac3f"
-					(reference "#PWR028")
-					(unit 1)
-				)
-			)
-		)
-	)
-	(symbol
 		(lib_id "Device:D")
 		(at 92.71 60.96 90)
@@
 					(unit 1)
 				)
+			)
+		)
+	)
+	(symbol
+		(lib_id "PCM_SparkFun-PowerSymbol:3.3V")
+		(at 19.05 127 0)
+		(unit 1)
+		(body_style 1)
+		(exclude_from_sim no)
+		(in_bom yes)
+		(on_board yes)
+		(in_pos_files yes)
+		(dnp no)
+		(fields_autoplaced yes)
+		(property "Reference" "#PWR028"
+			(at 19.05 130.81 0)
+			(hide yes)
+			(show_name no)
+			(do_not_autoplace no)
+			(effects
+				(font
+					(size 1.27 1.27)
+				)
+			)
+		)
+		(property "Value" "+3.3V"
+			(at 19.05 123.19 0)
+			(show_name no)
+			(do_not_autoplace yes)
+			(effects
+				(font
+					(size 1.27 1.27)
+				)
+			)
+		)
+		(property "Footprint" ""
+			(at 19.05 127 0)
+			(hide yes)
+			(show_name no)
+			(do_not_autoplace no)
+			(effects
+				(font
+					(size 1.27 1.27)
+				)
+			)
+		)
+		(property "Datasheet" ""
+			(at 19.05 127 0)
+			(hide yes)
+			(show_name no)
+			(do_not_autoplace no)
+			(effects
+				(font
+					(size 1.27 1.27)
+				)
+			)
+		)
+		(property "Description" "Power symbol creates a global label with name \"3.3V\""
+			(at 19.05 133.35 0)
+			(hide yes)
+			(show_name no)
+			(do_not_autoplace no)
+			(effects
+				(font
+					(size 1.27 1.27)
+				)
+			)
+		)
+		(pin "1"
+		)
+		(instances
+			(project "mitten40percent"
+				(path "/4d97bcd4-b797-40db-b476-9202db9dac3f"
+					(reference "#PWR028")
+					(unit 1)
+				)

Commit message: finalized routing
Connections:
- net C0: now also U1.4 (PC15); no longer U1.31 (PA10)
- net C1: now also U1.3 (PC14); no longer U1.30 (PA9)
- net C10: now also U1.26 (PB13); no longer U1.14 (PA4)
- net C11: now also U1.25 (PB12); no longer U1.13 (PA3)
- net C2: now also U1.2 (PC13); no longer U1.29 (PA8)
- net C3: now also U1.12 (PA2); no longer U1.28 (PB15)
- net C4: now also U1.17 (PA7); no longer U1.27 (PB14)
- net C5: now also U1.16 (PA6); no longer U1.26 (PB13)
- net C6: now also U1.15 (PA5); no longer U1.25 (PB12)
- net C7: now also U1.14 (PA4); no longer U1.17 (PA7)
- net C8: now also U1.13 (PA3); no longer U1.16 (PA6)
- net C9: now also U1.27 (PB14); no longer U1.15 (PA5)
- net JoystickSelect: now also U1.28 (PB15); no longer U1.38 (PA15)
- net JoystickX: now also U1.30 (PA9); no longer U1.34 (PA13)
- net JoystickY: now also U1.29 (PA8); no longer U1.37 (PA14)
Other:
- company: poo poo pee pee corporation -> bumbling idiots inc.
- moved on the sheet: C1, U1
