File: mitten40percentPCB/mitten40percent.kicad_pcb (KiCad board)
At the start: 2 copper layers, 114 parts, among them J2 I2C, J3 USB_C_Receptacle_USB2.0_16P, SW0 SW_Push, SW1 SW_Push_45deg, SW10 SW_Push_45deg, SW11 SW_Push_45deg, SW12 SW_Push_45deg, SW13 SW_Push_45deg, SW14 SW_Push_45deg, SW15 SW_Push_45deg, SW16 SW_Push_45deg, SW17 SW_Push_45deg, SW18 SW_Push_45deg, SW19 SW_Push_45deg, SW2 SW_Push_45deg, SW20 SW_Push_45deg, SW21 SW_Push_45deg, SW22 SW_Push_45deg, SW23 SW_Push_45deg, SW24 SW_Push_45deg, SW25 SW_Push_45deg, SW26 SW_Push_45deg, SW27 SW_Push_45deg, SW28 SW_Push_45deg, SW29 SW_Push_45deg, SW3 SW_Push_45deg, SW30 SW_Push_45deg, SW31 SW_Push_45deg, SW32 SW_Push_45deg, SW33 SW_Push_45deg, SW34 SW_Push_45deg, SW35 SW_Push_45deg, SW36 SW_Push_45deg, SW37 SW_Push_45deg, SW38 SW_Push_45deg, SW39 SW_Push_45deg, SW4 SW_Push_45deg, SW40 SW_Push_45deg, SW41 SW_Push_45deg, SW42 SW_Push_45deg, SW43 SW_Push_45deg, SW44 SW_Push_45deg, SW45 SW_Push_45deg, SW46 SW_Push_45deg, SW48 Joystick, SW5 SW_Push_45deg, SW6 SW_Push_45deg, SW7 SW_Push_45deg, SW8 SW_Push_45deg, SW9 SW_Push_45deg, U1 STM32F072CBT6, U2 USBLC6-2SC6, U3 XC6206PxxxMR

Commit message: finished wiring individual components (stm32, usb-c port, reset button), routed the matrix to the mcu
Parts:
- C1, C4, C5, C6, C7, R1, SW0: moved to B.Cu
- J2: footprint PCM_SparkFun-Connector:1x04_P2.54mm -> Display:ER_OLEDM0.91_1x-I2C
- moved SW48 237.5 mm to (31.8, 97.9)
- moved J2 230.0 mm to (35.4, 71.6), turned to 180 degrees
- moved R3 125.9 mm to (36.1, 16.4), turned to -90 degrees
- moved R2 123.0 mm to (39.2, 16.4), turned to -90 degrees
- moved J3 121.1 mm to (37.9, 10.2), turned to 180 degrees
- moved U2 118.6 mm to (37.0, 21.2), turned to 90 degrees
- moved U3 108.1 mm to (36.3, 30.7), turned to 90 degrees
- moved C10 107.4 mm to (35.8, 27.9), turned to 180 degrees
- moved F1 107.0 mm to (35.5, 26.5)
- moved C11 103.9 mm to (36.8, 33.3), turned to 180 degrees
- moved C9 92.8 mm to (36.7, 51.1), turned to 90 degrees
- moved C8 92.8 mm to (35.7, 51.1), turned to 90 degrees
- moved U1 91.3 mm to (32.9, 57.2)
- moved C3 90.8 mm to (26.7, 54.4)
- moved C4 88.9 mm to (26.7, 53.3), turned to 180 degrees
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Connections:
- U1 pad 12: /C4 -> unconnected-(U1-PA2-Pad12)
- U1 pad 13: /C5 -> /C11
- U1 pad 14: /C6 -> /C10
- U1 pad 15: /C7 -> /C9
- U1 pad 17: /C9 -> /C7
- U1 pad 25: /C0 -> /C6
- U1 pad 26: /C1 -> /C5
- U1 pad 27: /C2 -> /C4
- U1 pad 29: /C10 -> /C2
- U1 pad 30: /C11 -> /C1
- U1 pad 31: unconnected-(U1-PA10-Pad31) -> /C0
Routing:
- net /C11: track 0.00 -> 321.2 mm
- net /R3: track 0.00 -> 288.3 mm
- net /R2: track 0.00 -> 272.4 mm
- net /R1: track 0.00 -> 257.1 mm
- net /R0: track 0.00 -> 257.0 mm
- net /C10: track 0.00 -> 243.5 mm
- net /C9: track 0.00 -> 222.9 mm
- net /C7: track 0.00 -> 219.8 mm
- net /C6: track 0.00 -> 213.8 mm
- net /C8: track 0.00 -> 202.3 mm
- net /C4: track 0.00 -> 173.9 mm
- net /C5: track 0.00 -> 170.9 mm
- net /C2: track 0.00 -> 130.1 mm
- net /C1: track 0.00 -> 110.1 mm
- net /C3: track 0.00 -> 92.9 mm
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
Commit message: finished routing and ground fill, now on to santiy checks
Parts:
- moved R1 110.9 mm to (44.1, 64.8), turned to 180 degrees
- moved C11 23.2 mm to (42.6, 55.8)
- moved C10 23.2 mm to (41.7, 50.4)
- moved F1 23.2 mm to (41.4, 49.0)
- moved R2 23.2 mm to (45.1, 38.8)
- moved U2 23.2 mm to (42.9, 43.7)
- moved R3 23.2 mm to (42.0, 38.8)
- moved U3 23.2 mm to (42.2, 53.2)
- moved J3 22.5 mm to (43.7, 31.9)
- moved SW0 18.3 mm to (42.1, 68.5), turned to 0 degrees
- moved C4 1.88 mm to (28.6, 53.1), turned to 90 degrees
- moved C3 1.48 mm to (27.4, 53.1), turned to 90 degrees
- moved C8 1.39 mm to (36.6, 52.2), turned to -90 degrees
- moved C9 1.39 mm to (37.6, 52.2), turned to -90 degrees
- moved SW48 0.62 mm to (31.7, 97.3), turned to -90 degrees
Connections:
- J2 pad 2: +3V3 -> +3.3V
Routing:
- net +3.3V: track 53.6 -> 127.5 mm
- net /C3: track 92.9 -> 150.0 mm
- net /C8: track 202.3 -> 258.8 mm
- net /C9: track 222.9 -> 279.4 mm
- net /C10: track 243.5 -> 300.0 mm
- net /JoystickX: track 0.00 -> 51.1 mm, vias 0 -> 2
- net /JoystickSelect: track 0.00 -> 42.6 mm, vias 0 -> 2
- net /JoystickY: track 0.00 -> 37.7 mm
- net GND: track 11.1 -> 35.4 mm, vias 0 -> 7
- net /SCL: track 0.00 -> 18.0 mm, vias 0 -> 2
- net /SDA: track 0.00 -> 17.9 mm
- net /MCU_D-: track 0.00 -> 16.3 mm, vias 0 -> 1
- net /MCU_D+: track 0.00 -> 14.2 mm, vias 0 -> 1
- net /BOOT0: track 9.52 -> 20.3 mm, vias 0 -> 2
- net VBUS: track 15.1 -> 23.1 mm, vias 2 -> 3
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- added copper zone on B.Cu, net GND
- added copper zone on F.Cu, net GND
Other:
- board outline added: 263.3 x 87.2 mm

Commit message: finalized routing
Parts:
- C10, C11, F1, J3, R2, R3, U2, U3: moved to B.Cu
- moved R1 37.7 mm to (20.8, 35.1)
- moved SW0 34.2 mm to (25.1, 38.8)
- moved C2 19.8 mm to (43.2, 45.0), turned to 90 degrees
- moved C5 15.1 mm to (36.5, 45.1), turned to 90 degrees
- moved C1 13.9 mm to (40.3, 51.5), turned to 180 degrees
- moved C6 13.7 mm to (40.3, 52.6), turned to 0 degrees
- moved C7 13.7 mm to (40.3, 53.7), turned to 0 degrees
- moved C11 11.0 mm to (44.5, 44.9), turned to 90 degrees
- moved C10 10.5 mm to (47.3, 41.5), turned to 0 degrees
- moved C9 10.4 mm to (28.8, 46.6), turned to 0 degrees
- moved U3 10.2 mm to (46.9, 44.1)
- moved F1 9.89 mm to (46.1, 40.3)
- moved C8 9.04 mm to (28.8, 47.7), turned to 0 degrees
- moved U2 8.31 mm to (35.2, 40.5), turned to 0 degrees
- moved U1 5.92 mm to (33.7, 51.3), turned to 180 degrees
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Connections:
- U1 pad 12: unconnected-(U1-PA2-Pad12) -> /C3
- U1 pad 13: /C11 -> /C8
- U1 pad 14: /C10 -> /C7
- U1 pad 15: /C9 -> /C6
- U1 pad 16: /C8 -> /C5
- U1 pad 17: /C7 -> /C4
- U1 pad 2: unconnected-(U1-PC13-Pad2) -> /C2
- U1 pad 25: /C6 -> /C11
- U1 pad 26: /C5 -> /C10
- U1 pad 27: /C4 -> /C9
- U1 pad 28: /C3 -> /JoystickSelect
- U1 pad 29: /C2 -> /JoystickY
- U1 pad 3: unconnected-(U1-PC14-Pad3) -> /C1
- U1 pad 30: /C1 -> /JoystickX
- U1 pad 31: /C0 -> unconnected-(U1-PA10-Pad31)
- U1 pad 34: /JoystickX -> unconnected-(U1-PA13-Pad34)
- U1 pad 37: /JoystickY -> unconnected-(U1-PA14-Pad37)
- U1 pad 38: /JoystickSelect -> unconnected-(U1-PA15-Pad38)
- U1 pad 4: unconnected-(U1-PC15-Pad4) -> /C0
Routing:
- net +3.3V: track 127.5 -> 163.6 mm, vias 6 -> 8
- net /R3: track 288.4 -> 311.2 mm, vias 0 -> 2
- net /R2: track 272.5 -> 294.4 mm, vias 0 -> 2
- net /R1: track 257.1 -> 278.0 mm, vias 0 -> 2
- net /C8: track 258.8 -> 240.9 mm
- net /C7: track 219.2 -> 203.3 mm
- net /BOOT0: track 20.3 -> 35.4 mm
- net /C3: track 150.0 -> 136.5 mm
- net /C9: track 279.4 -> 292.4 mm
- net /C2: track 130.1 -> 119.5 mm, vias 0 -> 1
- net /C10: track 300.0 -> 310.3 mm
- net /C1: track 110.2 -> 100.3 mm, vias 0 -> 1
- net GND: track 35.4 -> 26.1 mm, vias 7 -> 8
- net /C0: track 89.3 -> 81.0 mm, vias 2 -> 1
- net /JoystickSelect: track 42.6 -> 50.5 mm, vias 2 -> 0
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Other:
- board text added: "C1"
- board text added: "C2"
- board text added: "C3"
- board text added: "C4"
- board text added: "C6"
- board text added: "C7"
- board text added: "C8"
- board text added: "C9"

Commit message: added silkscreen art
Parts:
- added G***: LOGO, coolArt:LargeYAK-130, B.Cu at (160.9, 92.3)
Other:
- board text added: "by louiNgn"
- board text added: "mitten40"
