File: mitten40percentPCB/mitten40percent.kicad_pcb (KiCad board)
At the start: 2 copper layers, 263.3 x 87.2 mm, 115 parts, among them J2 I2C, J3 USB_C_Receptacle_USB2.0_16P, SW0 SW_Push, SW1 SW_Push_45deg, SW10 SW_Push_45deg, SW11 SW_Push_45deg, SW12 SW_Push_45deg, SW13 SW_Push_45deg, SW14 SW_Push_45deg, SW15 SW_Push_45deg, SW16 SW_Push_45deg, SW17 SW_Push_45deg, SW18 SW_Push_45deg, SW19 SW_Push_45deg, SW2 SW_Push_45deg, SW20 SW_Push_45deg, SW21 SW_Push_45deg, SW22 SW_Push_45deg, SW23 SW_Push_45deg, SW24 SW_Push_45deg, SW25 SW_Push_45deg, SW26 SW_Push_45deg, SW27 SW_Push_45deg, SW28 SW_Push_45deg, SW29 SW_Push_45deg, SW3 SW_Push_45deg, SW30 SW_Push_45deg, SW31 SW_Push_45deg, SW32 SW_Push_45deg, SW33 SW_Push_45deg, SW34 SW_Push_45deg, SW35 SW_Push_45deg, SW36 SW_Push_45deg, SW37 SW_Push_45deg, SW38 SW_Push_45deg, SW39 SW_Push_45deg, SW4 SW_Push_45deg, SW40 SW_Push_45deg, SW41 SW_Push_45deg, SW42 SW_Push_45deg, SW43 SW_Push_45deg, SW44 SW_Push_45deg, SW45 SW_Push_45deg, SW46 SW_Push_45deg, SW48 Joystick, SW5 SW_Push_45deg, SW6 SW_Push_45deg, SW7 SW_Push_45deg, SW8 SW_Push_45deg, SW9 SW_Push_45deg, U1 STM32F072CBT6, U2 USBLC6-2SC6, U3 XC6206PxxxMR

Commit message: fixed up a potential clearance issue between joystick and keycaps, fingers crossed
Parts:
- moved D20 89.8 mm to (258.4, 127.7)
- moved D32 89.8 mm to (258.4, 146.8)
- moved D8 89.8 mm to (258.4, 108.7)
- moved SW11 89.8 mm to (310.4, 104.7)
- moved SW23 89.8 mm to (310.4, 123.7)
- moved SW35 89.8 mm to (310.4, 142.8)
- moved SW45 89.8 mm to (310.4, 161.8)
- moved C1 89.8 mm to (101.9, 116.8)
- moved C11 89.8 mm to (106.2, 110.3)
- moved C5 89.8 mm to (98.1, 110.5)
- moved C6 89.8 mm to (101.9, 117.9)
- moved C7 89.8 mm to (101.9, 119.1)
- moved C8 89.8 mm to (90.4, 113.0)
- moved D1 89.8 mm to (125.0, 108.7)
- moved D10 89.8 mm to (296.4, 108.7)
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Routing:
- net /JoystickSelect: track 50.5 -> 40.9 mm
- net /JoystickY: track 40.3 -> 32.9 mm
- net +3.3V: track 163.6 -> 158.8 mm
- net /JoystickX: track 51.7 -> 47.8 mm
Other:
- board size 263.3 x 87.2 mm -> 278.2 x 87.2 mm
